Commit message: fixed urdf added joints

File: src/car_support/urdf/car.urdf (robot description, URDF)
Before this commit: robot car, 5 links, 4 joints
Links:
- link FLwheel: geometry collision cylinder length=0.06 radius=0.125; visual cylinder length=0.06 radius=0.125
- link FRwheel: geometry collision cylinder length=0.06 radius=0.125; visual cylinder length=0.06 radius=0.125
- link RLwheel: geometry collision cylinder length=0.06 radius=0.125; visual cylinder length=0.06 radius=0.125
- link RRwheel: geometry collision cylinder length=0.06 radius=0.125; visual cylinder length=0.06 radius=0.125

Commit message: fixed urdf

File: src/car_support/urdf/car.urdf (robot description, URDF)
Before this commit: robot car, 5 links, 4 joints
Joints:
- joint FLw2Body: axis (none) -> 1 0 0; origin (none) -> xyz=0.16 0.25 0 rpy=0 0 0
- joint FRw2Body: axis (none) -> 1 0 0; origin (none) -> xyz=-0.16 0.25 0 rpy=0 0 0
- joint RLw2Body: axis (none) -> 1 0 0; origin (none) -> xyz=0.16 -0.25 0 rpy=0 0 0
- joint RRw2Body: axis (none) -> 1 0 0; origin (none) -> xyz=-0.16 -0.25 0 rpy=0 0 0
